File: CompactMP3/CompactMP3.kicad_pcb (KiCad board)
At the start: 2 copper layers, 14 x 12 mm, 24 parts, among them J1 USB_A_PCB_Edge_receptacle, Q1 AO3401A, U1 LP5907MFX-3.3/NOPB, U10 CH572D, U2 ES8316, U3 RP2354A, U4 TCR2EF33_LMCT, U5 TP4057_C725791, U8 ANT3216LL00R2400A, Y3 32mhz

Commit message: alot of work worked on, layout started
Parts:
- added C10: 1uF, CHXXX:0402, F.Cu at (182.3, 142.5)
- added C15: 1uF, CHXXX:0402, F.Cu at (179.1, 148.5)
- added C16: 10uF, Footprint:0603, F.Cu at (38.2, 106.1)
- added C17: 10uF, Footprint:0603, F.Cu at (42.4, 91.6)
- added C18: 0.1uF, CHXXX:0402, F.Cu at (58.2, 96.2)
- added C19: 10uF, Footprint:0603, F.Cu at (42.4, 94.0)
- added C20: 1uF, CHXXX:0402, F.Cu at (186.9, 140.4)
- added C21: 1uF, CHXXX:0402, F.Cu at (183.1, 144.2)
- added C22: 0.1uF, CHXXX:0402, F.Cu at (183.1, 143.3)
- added C23: 1uF, CHXXX:0402, F.Cu at (173.8, 142.4)
- added C24: 1uF, CHXXX:0402, F.Cu at (176.6, 144.9)
- added C25: 12pF, CHXXX:0402, F.Cu at (61.4, 93.9)
- added C26: 4.7uF, Footprint:0603, F.Cu at (42.4, 96.4)
- added C27: 12pF, CHXXX:0402, F.Cu at (61.4, 96.2)
- added C28: 4.7uF, Footprint:0603, F.Cu at (42.4, 98.8)
- added C29: 4.7uF, Footprint:0603, F.Cu at (42.4, 101.2)
- added C3: 1uF, CHXXX:0402, F.Cu at (185.1, 140.5)
- added C30: 4.7uF, Footprint:0603, F.Cu at (42.4, 103.6)
- added C33: 0.1uF, CHXXX:0402, F.Cu at (61.4, 98.6)
- added C34: 0.1uF, CHXXX:0402, F.Cu at (61.4, 100.9)
- added C35: 0.1uF, CHXXX:0402, F.Cu at (61.4, 103.3)
- added C36: 0.1uF, CHXXX:0402, F.Cu at (61.4, 105.6)
- added C37: 0.1uF, CHXXX:0402, F.Cu at (64.5, 91.5)
- added C38: 0.1uF, CHXXX:0402, F.Cu at (64.5, 93.9)
- added C39: 0.1uF, CHXXX:0402, F.Cu at (64.5, 96.2)
- added C4: 1uF, CHXXX:0402, F.Cu at (180.9, 139.8)
- added C40: 0.1uF, CHXXX:0402, F.Cu at (64.5, 98.6)
- added C41: 0.1uF, CHXXX:0402, F.Cu at (64.5, 100.9)
- added C42: 0.1uF, CHXXX:0402, F.Cu at (64.5, 103.3)
- added C43: 0.1uF, CHXXX:0402, F.Cu at (64.5, 105.6)
- added C5: 0.1uF, CHXXX:0402, F.Cu at (34.0, 101.2)
- added C6: 1uF, CHXXX:0402, F.Cu at (181.3, 142.5)
- added C7: 1uF, CHXXX:0402, F.Cu at (177.6, 147.3)
- added C8: 1uF, CHXXX:0402, F.Cu at (186.1, 139.0)
- added C9: 1uF, CHXXX:0402, F.Cu at (182.5, 148.6)
- added CN1: B2B-PH-K-S(LF)(SN), EasyEDA:CONN-TH_B2B-PH-K-S, F.Cu at (74.8, 136.3)
- added CN2: PJ-320D, EasyEDA:AUDIO-SMD_PJ-320D-1, F.Cu at (193.8, 144.7)
- added Card1: TF PUSH, EasyEDA:TF-SMD_TF-PUSH, F.Cu at (147.2, 120.8)
- added J2: USB4105-GF-A, Footprint:usbc, F.Cu at (147.2, 91.1)
- added J3: screen, Footprint:PinHeader_01x04_P2.54mm_Vertical_THT_D1mm, F.Cu at (41.9, 180.8)
- added L1: 3.3uH, Footprint:0603, F.Cu at (42.4, 106.1)
- added Q2: AO3401A, EasyEDA:SOT-23_L2.9-W1.3-P1.90-LS2.4-BR, F.Cu at (76.1, 96.7)
- added R10: 4.7k, Footprint:0603, F.Cu at (122.6, 155.1)
- added R11: 4.7k, Footprint:0603, F.Cu at (122.6, 153.7)
- added R12: 1.5k, Footprint:0603, F.Cu at (50.8, 103.6)
- added R13: 5.1k, Footprint:0603, F.Cu at (50.8, 106.1)
- added R14: 5.1k, Footprint:0603, F.Cu at (55.0, 91.6)
- added R15: 1.5k, Footprint:0603, F.Cu at (55.0, 94.0)
- added R16: 33, Footprint:0603, F.Cu at (55.0, 96.4)
- added R17: 27, Footprint:0603, F.Cu at (55.0, 98.8)
- added R18: 27, Footprint:0603, F.Cu at (55.0, 101.2)
- added R19: 1.5k, Footprint:0603, F.Cu at (55.0, 103.6)
- added R3: 100k, Footprint:0603, F.Cu at (46.6, 98.8)
- added R4: 100k, Footprint:0603, F.Cu at (46.6, 101.2)
- added R5: 100k, Footprint:0603, F.Cu at (46.6, 103.6)
- added R6: 47k, Footprint:0603, F.Cu at (46.6, 106.1)
- added R7: 47k, Footprint:0603, F.Cu at (50.8, 91.6)
- added R8: 33, Footprint:0603, F.Cu at (186.9, 141.9)
- added R9: 33, Footprint:0603, F.Cu at (186.9, 145.8)
- added S1: TL3365AF180QG, Footprint:button, F.Cu at (70.5, 92.7)
- added S2: TL3365AF180QG, Footprint:button, F.Cu at (70.5, 97.5)
- added S3: TL3365AF180QG, Footprint:button, F.Cu at (70.5, 102.2)
- added SW1: SKRTLAE010, EasyEDA:KEY-SMD_SKRTLAE010, F.Cu at (196.9, 107.5)
- added SW2: SKRTLAE010, EasyEDA:KEY-SMD_SKRTLAE010, F.Cu at (196.9, 114.1)
- added SW3: SKRTLAE010, EasyEDA:KEY-SMD_SKRTLAE010, F.Cu at (197.3, 120.6)
- added SW4: SKRTLAE010, EasyEDA:KEY-SMD_SKRTLAE010, F.Cu at (196.9, 126.9)
- added SW5: SKRTLAE010, EasyEDA:KEY-SMD_SKRTLAE010, F.Cu at (196.9, 134.0)
- added TP10: GND, Footprint:SMD_TP_0.8mm, F.Cu at (73.9, 124.8)
- added TP11: MOSI, Footprint:SMD_TP_0.8mm, F.Cu at (76.6, 179.3)
- added TP12: MISO, Footprint:SMD_TP_0.8mm, F.Cu at (85.2, 179.3)
- added TP13: SCK, Footprint:SMD_TP_0.8mm, F.Cu at (89.6, 179.3)
- added TP14: SCS, Footprint:SMD_TP_0.8mm, F.Cu at (80.9, 179.3)
- added TP15: SD_PWR, Footprint:SMD_TP_0.8mm, F.Cu at (75.7, 121.2)
- added TP16: PWR_IN, Footprint:SMD_TP_0.8mm, F.Cu at (93.9, 179.3)
- added TP17: DSDIN, Footprint:SMD_TP_0.8mm, F.Cu at (174.0, 145.9)
- added TP18: DLRCK, Footprint:SMD_TP_0.8mm, F.Cu at (173.3, 146.7)
- added TP19: SCLK, Footprint:SMD_TP_0.8mm, F.Cu at (174.8, 145.3)
- added TP20: CDATA, Footprint:SMD_TP_0.8mm, F.Cu at (178.7, 142.2)
- added TP21: CCLK, Footprint:SMD_TP_0.8mm, F.Cu at (177.6, 143.2)
- added TP22: MCLK, Footprint:SMD_TP_0.8mm, F.Cu at (176.3, 143.6)
- added TP23: 1.8V, Footprint:SMD_TP_0.8mm, F.Cu at (179.6, 149.7)
- added TP24: 3.3V, Footprint:SMD_TP_0.8mm, F.Cu at (175.3, 144.1)
- added TP25: 3.3V Clean, Footprint:SMD_TP_0.8mm, F.Cu at (183.2, 141.8)
- added TP26: VSYS, Footprint:SMD_TP_0.8mm, F.Cu at (185.1, 137.8)
- added TP27: GND, Footprint:SMD_TP_0.8mm, F.Cu at (183.8, 146.8)
- added TP30: 1/2 BATTERY, Footprint:SMD_TP_0.8mm, F.Cu at (79.3, 123.0)
- added TP31: VSYS, Footprint:SMD_TP_0.8mm, F.Cu at (79.3, 124.8)
- added TP32: POWER IN, Footprint:SMD_TP_0.8mm, F.Cu at (79.3, 126.6)
- added TP33: BATTERY +, Footprint:SMD_TP_0.8mm, F.Cu at (79.3, 128.4)
- added TP5: CS, Footprint:SMD_TP_0.8mm, F.Cu at (72.1, 128.4)
- added TP6: MOSI, Footprint:SMD_TP_0.8mm, F.Cu at (72.1, 130.2)
- added TP7: SCK, Footprint:SMD_TP_0.8mm, F.Cu at (72.1, 132.0)
- added TP8: MISO, Footprint:SMD_TP_0.8mm, F.Cu at (73.9, 121.2)
- added TP9: IN, Footprint:SMD_TP_0.8mm, F.Cu at (73.9, 123.0)
- added U6: TPMIC5365-1.8YC5, EasyEDA:SOT-323-5_L2.1-W1.3-P0.65-LS2.1-BL, F.Cu at (176.5, 149.1)
- added X1: XTM32012000JT00351006, EasyEDA:CRYSTAL-SMD_4P-L3.2-W2.5-BL, F.Cu at (52.4, 134.1)
- C1, C14, C2: footprint Footprint:0603 -> CHXXX:0402
- C11, C12: footprint Footprint:C_0603 -> Footprint:0603
- D1: footprint EasyEDA:SMA_L4.3-W2.6-LS5.0-RD -> EasyEDA:SOD-123FL_L2.8-W1.8-LS3.7-RD
- TP3: value CH572D- -> 3.3V
- TP4: value CH572D- -> GND
- moved U2 138.3 mm to (180.3, 145.3), turned to -90 degrees
- moved C11 133.6 mm to (20.3, 179.3)
- moved C12 129.9 mm to (24.6, 179.7)
- moved U1 129.7 mm to (183.0, 139.3), turned to 90 degrees
- moved U8 127.3 mm to (72.2, 180.1)
- moved C13 122.5 mm to (28.9, 179.7)
- moved Y3 117.8 mm to (33.5, 180.2)
- moved C14 115.9 mm to (50.2, 179.3)
- moved L2 115.8 mm to (37.6, 179.7)
- moved U10 114.8 mm to (45.3, 159.8), turned to -90 degrees
- moved J1 114.5 mm to (69.3, 163.3), turned to 135 degrees
- moved TP1 114.5 mm to (59.2, 179.3)
- moved TP2 113.2 mm to (54.9, 179.3)
- moved TP3 110.4 mm to (67.9, 179.3)
- moved TP4 108.8 mm to (63.6, 179.3)
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Connections:
- net BAT+ renamed BATTERY+
- C1 pad 2: PWR_5V -> VSYS
- C13 pad 1: PWR_3V3 -> V33
- C14 pad 1: PWR_3V3 -> V33
- C2 pad 1: PWR_3V3 -> V33
- TP3 pad 1: PWR_GND -> V33
- TP4 pad 1: unconnected-(TP4-Pad1) -> PWR_GND
- U1 pad 1: PWR_5V -> VSYS
- U1 pad 3: unconnected-(U1-EN-Pad3) -> VSYS
- U1 pad 5: unconnected-(U1-OUT-Pad5) -> AVDD
- U10 pad 1: unconnected-(U10-PA3/T/R1/SCL2/SCK_/PWM3/CP0-Pad1) -> CH572_SCREEN_SCL
- U10 pad 13: unconnected-(U10-PA4/SCS/PWM4/TMR2-Pad13) -> CH572_SCS
- U10 pad 14: PA5 -> CH572_SCK
- U10 pad 15: PA6 -> CH572_MISO
- U10 pad 16: unconnected-(U10-PA7/MOSI/T4/PWM1/TMR/RST_/CP1-Pad16) -> CH572_MOSI
- U10 pad 20: unconnected-(U10-PA2/R/T1/SDA2/SCS_/PWM2/TMR1/CN-Pad20) -> CH572_SCREEN_SDA
- U10 pad 6: PWR_3V3 -> V33
- U10 pad 7: PWR_3V3 -> V33
- U10 pad 8: PWR_3V3 -> V33
- U2 pad 1: unconnected-(U2-CCLK-Pad1) -> CCLK
- U2 pad 13: unconnected-(U2-CPVSSP-Pad13) -> Net-(U2-CPVSSP)
- U2 pad 14: unconnected-(U2-CPVDD-Pad14) -> 1V8
- U2 pad 15: unconnected-(U2-CPTOP-Pad15) -> Net-(U2-CPTOP)
- U2 pad 16: unconnected-(U2-CPBOT-Pad16) -> Net-(U2-CPBOT)
- U2 pad 17: unconnected-(U2-CPGND-Pad17) -> PWR_GND
- U2 pad 18: unconnected-(U2-CPGNDREF-Pad18) -> PWR_GND
- U2 pad 19: unconnected-(U2-ROUT-Pad19) -> Net-(U2-ROUT)
- U2 pad 2: unconnected-(U2-MCLK-Pad2) -> MCLK
- U2 pad 20: unconnected-(U2-LOUT-Pad20) -> Net-(U2-LOUT)
- U2 pad 21: unconnected-(U2-DACVREF-Pad21) -> Net-(U2-DACVREF)
- U2 pad 22: unconnected-(U2-AVDD-Pad22) -> AVDD
- U2 pad 23: unconnected-(U2-AGND-Pad23) -> PWR_GND
- U2 pad 24: unconnected-(U2-ADCVREF-Pad24) -> Net-(U2-ADCVREF)
- U2 pad 25: unconnected-(U2-VMID-Pad25) -> Net-(U2-VMID)
- U2 pad 3: unconnected-(U2-DVDD-Pad3) -> V33
- U2 pad 31: unconnected-(U2-CE-Pad31) -> PWR_GND
- U2 pad 32: unconnected-(U2-CDATA-Pad32) -> CDATA
- U2 pad 33: unconnected-(U2-EP-Pad33) -> PWR_GND
- U2 pad 4: unconnected-(U2-PVDD-Pad4) -> V33
- U2 pad 5: unconnected-(U2-DGND-Pad5) -> PWR_GND
- U2 pad 6: unconnected-(U2-SCLK-Pad6) -> SCLK
- U2 pad 7: unconnected-(U2-DSDIN-Pad7) -> DSDIN
- U2 pad 8: unconnected-(U2-DLRCK-Pad8) -> DLRCK
- U3 pad 1: unconnected-(U3-IOVDD-Pad1) -> V33
- U3 pad 11: unconnected-(U3-IOVDD-Pad11) -> V33
- U3 pad 12: unconnected-(U3-GPIO8-Pad12) -> SD_MISO
- U3 pad 13: unconnected-(U3-GPIO9-Pad13) -> SD_CS
- U3 pad 14: unconnected-(U3-GPIO10-Pad14) -> SD_SCK
- U3 pad 15: unconnected-(U3-GPIO11-Pad15) -> SD_MOSI
- U3 pad 16: unconnected-(U3-GPIO12-Pad16) -> CDATA
- U3 pad 17: unconnected-(U3-GPIO13-Pad17) -> CCLK
- U3 pad 18: unconnected-(U3-GPIO14-Pad18) -> SCLK
- U3 pad 19: unconnected-(U3-GPIO15-Pad19) -> DLRCK
- U3 pad 2: unconnected-(U3-GPIO0-Pad2) -> CH572_MISO
- U3 pad 20: unconnected-(U3-IOVDD-Pad20) -> V33
- U3 pad 21: unconnected-(U3-XIN-Pad21) -> XIN
- U3 pad 22: unconnected-(U3-XOUT-Pad22) -> XOUT
- U3 pad 23: unconnected-(U3-DVDD-Pad23) -> V11
- U3 pad 26: unconnected-(U3-RUN-Pad26) -> RST
- U3 pad 27: unconnected-(U3-GPIO16-Pad27) -> DSDIN
- U3 pad 28: unconnected-(U3-GPIO17-Pad28) -> MCLK
- U3 pad 3: unconnected-(U3-GPIO1-Pad3) -> CH572_SCS
- U3 pad 30: unconnected-(U3-IOVDD-Pad30) -> V33
- U3 pad 32: unconnected-(U3-GPIO20-Pad32) -> PLAY
- U3 pad 33: unconnected-(U3-GPIO21-Pad33) -> VOLUME-
- U3 pad 34: unconnected-(U3-GPIO22-Pad34) -> UNSKIP
- U3 pad 35: unconnected-(U3-GPIO23-Pad35) -> VOLUME+
- U3 pad 36: unconnected-(U3-GPIO24-Pad36) -> SKIP
- U3 pad 38: unconnected-(U3-IOVDD-Pad38) -> V33
- U3 pad 39: unconnected-(U3-DVDD-Pad39) -> V11
- U3 pad 4: unconnected-(U3-GPIO2-Pad4) -> CH572_SCK
- U3 pad 40: unconnected-(U3-GPIO26_ADC0-Pad40) -> BATMON
- U3 pad 44: unconnected-(U3-ADC_AVDD-Pad44) -> V33
- U3 pad 45: unconnected-(U3-IOVDD-Pad45) -> V33
- U3 pad 46: unconnected-(U3-VREG_AVDD-Pad46) -> Net-(U3-VREG_AVDD)
- U3 pad 47: unconnected-(U3-VREG_PGND-Pad47) -> PWR_GND
- U3 pad 48: unconnected-(U3-VREG_LX-Pad48) -> Net-(U3-VREG_LX)
- U3 pad 49: unconnected-(U3-VREG_VIN-Pad49) -> V33
- U3 pad 5: unconnected-(U3-GPIO3-Pad5) -> CH572_MOSI
- U3 pad 50: unconnected-(U3-VREG_FB-Pad50) -> V11
- U3 pad 51: unconnected-(U3-USB_DM-Pad51) -> Net-(U3-USB_DM)
- U3 pad 52: unconnected-(U3-USB_DP-Pad52) -> Net-(U3-USB_DP)
- U3 pad 53: unconnected-(U3-USB_OTP_VDD-Pad53) -> V33
- U3 pad 54: unconnected-(U3-QSPI_IOVDD-Pad54) -> V33
- U3 pad 6: unconnected-(U3-DVDD-Pad6) -> V11
- U3 pad 60: unconnected-(U3-QSPI_SS-Pad60) -> Net-(U3-QSPI_SS)
- U3 pad 61: unconnected-(U3-EP-Pad61) -> PWR_GND
- U3 pad 7: unconnected-(U3-GPIO4-Pad7) -> CH572_RST
- U3 pad 8: unconnected-(U3-GPIO5-Pad8) -> SD_DETECT
- U3 pad 9: unconnected-(U3-GPIO6-Pad9) -> SD_EN
- U4 pad 1: PWR_5V -> VSYS
- U4 pad 3: PWR_5V -> VSYS
- U4 pad 5: PWR_3V3 -> V33
Routing:
- net PWR_GND: track 0.00 -> 29.4 mm, vias 0 -> 16
- net VSYS: track 0.00 -> 9.81 mm
- net 1V8: track 0.00 -> 7.62 mm
- net Net-(U2-DACVREF): track 0.00 -> 7.40 mm
- net V33: track 0.00 -> 7.12 mm
- net Net-(U2-LOUT): track 0.00 -> 6.61 mm
- net AVDD: track 0.00 -> 6.29 mm
- net DLRCK: track 0.00 -> 5.02 mm
- net DSDIN: track 0.00 -> 4.38 mm
- net Net-(U2-ROUT): track 0.00 -> 4.03 mm
- net SCLK: track 0.00 -> 3.58 mm
- net MCLK: track 0.00 -> 2.70 mm
- net ROUT: track 0.00 -> 2.56 mm
- net LOUT: track 0.00 -> 2.54 mm
- net Net-(U2-CPBOT): track 0.00 -> 2.51 mm
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- added copper zone on B.Cu, net PWR_GND
Other:
- board size 14 x 12 mm -> 181.1 x 88.9 mm
- copper layers 2 -> 4

Commit message: more work, ch572d section start (not done
Parts:
- J1: moved to B.Cu
- moved TP16 50.9 mm to (48.5, 156.3)
- moved TP11 45.3 mm to (37.8, 155.9)
- moved TP12 45.3 mm to (46.5, 155.9)
- moved TP13 45.3 mm to (50.8, 155.9)
- moved TP14 45.3 mm to (42.2, 155.9)
- moved U3 44.2 mm to (84.3, 151.6)
- moved J3 29.6 mm to (29.6, 153.8), turned to 90 degrees
- moved U8 29.5 mm to (45.8, 167.2)
- moved TP3 26.0 mm to (46.3, 164.9), turned to 180 degrees
- moved C11 24.8 mm to (41.5, 166.4), turned to 180 degrees
- moved C12 24.6 mm to (41.5, 161.8), turned to 180 degrees
- moved C13 24.5 mm to (46.5, 162.6)
- moved Y3 22.8 mm to (42.1, 159.1), turned to 180 degrees
- moved TP1 22.0 mm to (48.3, 160.3)
- moved TP4 21.6 mm to (47.5, 164.9)
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Routing:
- net PWR_IN: track 0.00 -> 15.9 mm, vias 0 -> 1
- net VSYS: track 9.81 -> 21.5 mm, vias 0 -> 2
- net D-: track 0.00 -> 10.6 mm, vias 0 -> 1
- net D+: track 0.00 -> 10.3 mm, vias 0 -> 1
- net V33: track 7.12 -> 11.9 mm, vias 0 -> 2
- net Net-(C11-Pad1): track 0.00 -> 3.97 mm
- net Net-(U10-ANT): track 0.00 -> 3.83 mm
- net PWR_GND: track 29.4 -> 32.7 mm, vias 16 -> 41
- net Net-(U10-XO): track 0.00 -> 2.76 mm
- net Net-(U10-XI): track 0.00 -> 1.29 mm
- added copper zone on In1.Cu, net PWR_GND
- added copper zone on In2.Cu, net V33

Commit message: more work, barely any
Parts:
- moved J2 46.0 mm to (192.9, 95.9)
- moved Card1 35.4 mm to (176.2, 100.5), turned to 180 degrees
- moved TP13 7.30 mm to (43.9, 153.7)
- moved CN2 0.08 mm to (193.7, 144.7)
Routing:
- net PWR_GND: track 32.7 -> 38.1 mm
- net Net-(U2-CPTOP): track 1.15 -> 1.79 mm

Commit message: a buncha changes, nearing done but still time to work
Parts:
- moved J3 194.9 mm to (211.7, 84.3)
- moved Y3 141.7 mm to (176.6, 114.6), turned to 90 degrees
- moved C12 140.7 mm to (173.9, 114.0), turned to 90 degrees
- moved L2 138.3 mm to (171.6, 114.9), turned to 0 degrees
- moved C11 138.1 mm to (169.2, 113.9), turned to 90 degrees
- moved U10 137.2 mm to (175.9, 117.8), turned to 180 degrees
- moved C13 133.9 mm to (173.1, 119.0), turned to -90 degrees
- moved C14 133.4 mm to (171.9, 118.8), turned to -90 degrees
- moved TP2 133.2 mm to (174.5, 120.2), turned to -90 degrees
- moved TP1 133.1 mm to (175.4, 120.8), turned to -90 degrees
- moved TP3 132.7 mm to (170.7, 118.8), turned to 90 degrees
- moved U8 132.1 mm to (168.4, 118.2), turned to -90 degrees
- moved TP4 131.2 mm to (170.8, 119.9), turned to -90 degrees
- moved U3 105.6 mm to (186.5, 124.8)
- moved Q2 105.4 mm to (180.4, 112.2)
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Routing:
- net PWR_GND: track 38.1 -> 45.0 mm, vias 41 -> 46
- net Net-(Card1-VDD): track 0.00 -> 4.42 mm
- net CDATA: track 1.18 -> 4.87 mm
- net CCLK: track 1.10 -> 4.68 mm
- net V33: track 11.9 -> 14.2 mm, vias 2 -> 4

Commit message: worked on it
Parts:
- added C31: 0.1uF, CHXXX:0402, F.Cu at (191.3, 123.9)
- Card1: moved to B.Cu
- moved C5 165.9 mm to (199.9, 98.8), turned to 180 degrees
- moved C16 163.1 mm to (201.2, 99.3), turned to 90 degrees
- moved TP30 162.6 mm to (239.0, 92.4)
- moved TP33 160.6 mm to (235.7, 91.6)
- moved TP31 156.6 mm to (232.4, 91.6)
- moved R4 153.9 mm to (200.5, 103.6)
- moved TP32 153.8 mm to (229.1, 91.6)
- moved C17 153.5 mm to (195.6, 101.4), turned to -90 degrees
- moved R3 151.4 mm to (198.0, 96.8), turned to 180 degrees
- moved R1 149.8 mm to (196.3, 98.5), turned to 180 degrees
- moved R2 149.3 mm to (195.7, 103.9), turned to 180 degrees
- moved U5 139.5 mm to (198.5, 101.1)
- moved D1 134.8 mm to (199.1, 105.7), turned to 180 degrees
- moved CN1 133.7 mm to (204.4, 103.4), turned to 180 degrees
- moved Q1 124.0 mm to (199.1, 108.5), turned to -90 degrees
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Routing:
- net Net-(J2-CC1): track 0.00 -> 143.5 mm
- net PWR_GND: track 45.0 -> 135.3 mm, vias 46 -> 81
- net D+: track 10.3 -> 91.3 mm, vias 1 -> 2
- net Net-(Card1-DAT2): track 0.00 -> 50.4 mm, vias 0 -> 1
- net V11: track 0.00 -> 47.3 mm, vias 0 -> 2
- net V33: track 14.2 -> 45.6 mm, vias 4 -> 22
- net PWR_IN: track 15.9 -> 47.1 mm
- net XIN: track 0.00 -> 30.6 mm
- net Net-(R12-Pad1): track 0.00 -> 27.7 mm
- net Net-(U3-VREG_AVDD): track 0.00 -> 22.8 mm, vias 0 -> 2
- net XOUT: track 0.00 -> 22.3 mm
- net Net-(R15-Pad2): track 0.00 -> 20.4 mm
- net Net-(R19-Pad2): track 0.00 -> 20.1 mm
- net Net-(R7-Pad1): track 0.00 -> 18.4 mm
- net BATMON: track 0.00 -> 16.6 mm
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