File: CompactMP3/CompactMP3.kicad_sch (KiCad schematic)
At the start: 38 parts, among them CN1 B2B-PH-K-S(LF)(SN), J1 USB_A_PCB_Edge_receptacle, Q1 AO3401A, U1 LP5907MFX-3.3/NOPB, U10 CH572D, U2 ES8316, U3 RP2354A, U4 TCR2EF33_LMCT, U5 TP4057_C725791, U6 TPMIC5365-1.8YC5, U8 ANT3216LL00R2400A, Y3 32mhz

Commit message: alot of work worked on, layout started
Parts:
- added C16, C17, C19: 10uF, Footprint:0603, symbol fab:C_0603
- added C18, C22: 0.1uF, CHXXX:0402, symbol fab:C_0603
- added C20, C21, C23, C24: 1uF, CHXXX:0402, symbol fab:C_0603
- added C25, C27: 12pF, CHXXX:0402, symbol 0402:C_0402
- added C26, C28, C29, C30: 4.7uF, Footprint:0603, symbol fab:C_0603
- added C33, C34, C35, C36, C37, C38, C39, C40, C41, C42, C43: 0.1uF, CHXXX:0402, symbol 0402:C_0402
- added CN2: PJ-320D, EasyEDA:AUDIO-SMD_PJ-320D-1, symbol EasyEDA:PJ-320D
- added J2: USB4105-GF-A, Footprint:usbc, symbol usbc:USB4105-GF-A
- added J3: screen, Footprint:PinHeader_01x04_P2.54mm_Vertical_THT_D1mm, symbol fab:PinHeader_01x04_P2.54mm_Vertical_THT_D1mm
- added L1: 3.3uH, Footprint:0603, symbol 0603:L_0603
- added Q2: AO3401A, EasyEDA:SOT-23_L2.9-W1.3-P1.90-LS2.4-BR, symbol EasyEDA:AO3401A
- added R10, R11: 4.7k, Footprint:0603, symbol fab:R_0603
- added R12, R15, R19: 1.5k, Footprint:0603, symbol fab:R_0603
- added R13, R14: 5.1k, Footprint:0603, symbol fab:R_0603
- added R16, R8, R9: 33, Footprint:0603, symbol fab:R_0603
- added R17, R18: 27, Footprint:0603, symbol fab:R_0603
- added R5: 100k, Footprint:0603, symbol fab:R_0603
- added R6, R7: 47k, Footprint:0603, symbol fab:R_0603
- added S1, S2, S3: TL3365AF180QG, Footprint:button, symbol button:TL3365AF180QG
- added SW1, SW2, SW3, SW4, SW5: SKRTLAE010, EasyEDA:KEY-SMD_SKRTLAE010, symbol EasyEDA:SKRTLAE010
- added TP10, TP27: GND, Footprint:SMD_TP_0.8mm, symbol Testpoint:testpoint
- added TP11, TP6: MOSI, Footprint:SMD_TP_0.8mm, symbol Testpoint:testpoint
- added TP12, TP8: MISO, Footprint:SMD_TP_0.8mm, symbol Testpoint:testpoint
- added TP13, TP7: SCK, Footprint:SMD_TP_0.8mm, symbol Testpoint:testpoint
- added TP14: SCS, Footprint:SMD_TP_0.8mm, symbol Testpoint:testpoint
- added TP15: SD_PWR, Footprint:SMD_TP_0.8mm, symbol Testpoint:testpoint
- added TP16: PWR_IN, Footprint:SMD_TP_0.8mm, symbol Testpoint:testpoint
- added TP17: DSDIN, Footprint:SMD_TP_0.8mm, symbol Testpoint:testpoint
- added TP18: DLRCK, Footprint:SMD_TP_0.8mm, symbol Testpoint:testpoint
- added TP19: SCLK, Footprint:SMD_TP_0.8mm, symbol Testpoint:testpoint
- added TP20: CDATA, Footprint:SMD_TP_0.8mm, symbol Testpoint:testpoint
- added TP21: CCLK, Footprint:SMD_TP_0.8mm, symbol Testpoint:testpoint
- added TP22: MCLK, Footprint:SMD_TP_0.8mm, symbol Testpoint:testpoint
- added TP23: 1.8V, Footprint:SMD_TP_0.8mm, symbol Testpoint:testpoint
- added TP24: 3.3V, Footprint:SMD_TP_0.8mm, symbol Testpoint:testpoint
- added TP25: 3.3V Clean, Footprint:SMD_TP_0.8mm, symbol Testpoint:testpoint
- added TP26, TP31: VSYS, Footprint:SMD_TP_0.8mm, symbol Testpoint:testpoint
- added TP30: 1/2 BATTERY, Footprint:SMD_TP_0.8mm, symbol Testpoint:testpoint
- added TP32: POWER IN, Footprint:SMD_TP_0.8mm, symbol Testpoint:testpoint
- added TP33: BATTERY +, Footprint:SMD_TP_0.8mm, symbol Testpoint:testpoint
- added TP5: CS, Footprint:SMD_TP_0.8mm, symbol Testpoint:testpoint
- added TP9: IN, Footprint:SMD_TP_0.8mm, symbol Testpoint:testpoint
- added X1: XTM32012000JT00351006, EasyEDA:CRYSTAL-SMD_4P-L3.2-W2.5-BL, symbol EasyEDA:XTM32012000JT00351006
- C1, C14, C2, C5: footprint Footprint:0603 -> CHXXX:0402
- C10, C15, C3, C4, C6, C7, C8, C9: footprint fab:C_0603 -> CHXXX:0402
- C11, C12: footprint Footprint:C_0603 -> Footprint:0603
- D1: footprint EasyEDA:SMA_L4.3-W2.6-LS5.0-RD -> EasyEDA:SOD-123FL_L2.8-W1.8-LS3.7-RD
Connections:
- net PA5 is gone; now on net CH572_SCK: U10.14 (PA5/SCK/SCL3)
- net PA6 is gone; now on net CH572_MISO: U10.15 (PA6/MISO/R4/SDA3)
- net 1V8: now also TP23.1
- net AVDD: now also C21.1, C22.1, TP25.1
- net BATMON: now also U3.40 (GPIO26_ADC0), TP30.1
- net CCLK: now also U3.17 (GPIO13), R10.2, TP21.1
- net CDATA: now also U3.16 (GPIO12), R11.1, TP20.1
- net CH572_RST: now also U3.7 (GPIO4)
- net D+: now also S1.1, S1.2
- net MCLK: now also U3.28 (GPIO17), TP22.1
- net PWR_GND: now also Card1.10, Card1.11, Card1.12, Card1.13, Card1.6 (VSS), U2.18 (CPGNDREF), U3.47 (VREG_PGND), U3.61 (EP), U6.2 (GND), C16.2, C17.2, C18.2, C19.2, C20.1, C21.2, C22.2, C23.1, C24.1, C25.2, C26.2, C27.2, C28.1, C29.2, C30.1, C34.1, C35.1, C36.2, CN2.2, J2.A1_B12 (GND), J2.B1_A12 (GND__1), J2.SH1 (SHELL_GND), J2.SH2 (SHELL_GND__1), J2.SH3 (SHELL_GND__2), J2.SH4 (SHELL_GND__3), J3.1 (Pin_1), R13.2, R14.2, S2.1, S2.2, S3.1, S3.2, SW1.1, SW1.3, SW1.4, SW1.5, SW2.1, SW2.3, SW2.4, SW2.5, SW3.1, SW3.3, SW3.4, SW3.5, SW4.1, SW4.3, SW4.4, SW4.5, SW5.1, SW5.3, SW5.4, SW5.5, TP10.1, TP27.1, X1.2 (GND), X1.4 (GND)
- net PWR_IN: now also C17.1, J2.A4_B9 (VBUS), J2.B4_A9 (VBUS__1), TP16.1, TP32.1
- net SCLK: now also U3.18 (GPIO14), TP19.1
- net V33: now also U3.1 (IOVDD), U3.11 (IOVDD), U3.20 (IOVDD), U3.30 (IOVDD), U3.38 (IOVDD), U3.44 (ADC_AVDD), U3.45 (IOVDD), U3.49 (VREG_VIN), U3.53 (USB_OTP_VDD), U3.54 (QSPI_IOVDD), C19.1, C23.2, C24.2, C29.1, C33.1, C36.1, C37.1, C38.1, C39.1, C40.1, C41.1, C42.1, C43.1, J3.2 (Pin_2), Q2.2 (S), R10.1, R11.2, R12.2, R16.2, R5.1, TP24.1
- net VSYS: now also U6.3 (EN), TP26.1, TP31.1
- net at U2.19 (ROUT): now also R9.2
- net at U2.20 (LOUT): now also R8.2
- net at U2.21 (DACVREF): now also C20.2
- net DSDIN: now reaches U2.7 (DSDIN)
- net DSDIN: now also U3.27 (GPIO16), TP17.1
- net DLRCK: now reaches U2.8 (DLRCK)
- net DLRCK: now also U3.19 (GPIO15), TP18.1
- net SD_MISO: now reaches U3.12 (GPIO8)
- net SD_MISO: now also Card1.7 (DAT0), TP8.1
- net SD_CS: now reaches U3.13 (GPIO9)
- net SD_CS: now also Card1.2 (CD/DAT3), TP5.1
- net SD_SCK: now reaches U3.14 (GPIO10)
- net SD_SCK: now also Card1.5 (CLX), TP7.1
- net SD_MOSI: now reaches U3.15 (GPIO11)
- net SD_MOSI: now also Card1.3 (CMD), TP6.1
- net CH572_MISO: now reaches U3.2 (GPIO0)
- net CH572_MISO: now also TP12.1
- net XIN: now reaches U3.21 (XIN)
- net XIN: now also C25.1, X1.1
- net XOUT: now reaches U3.22 (XOUT)
- net XOUT: now also C27.1, X1.3
- net V11: now reaches U3.23 (DVDD)
- net V11: now also U3.39 (DVDD), U3.50 (VREG_FB), U3.6 (DVDD), C26.1, C30.2, C34.2, C35.2, L1.1
- net RST: now reaches U3.26 (RUN)
- net RST: now also R19.1
- net CH572_SCS: now reaches U3.3 (GPIO1)
- net CH572_SCS: now also U10.13 (PA4/SCS/PWM4/TMR2), TP14.1
- net PLAY: now reaches U3.32 (GPIO20)
- net PLAY: now also SW1.2
- net VOLUME-: now reaches U3.33 (GPIO21)
- net VOLUME-: now also SW3.2
- net UNSKIP: now reaches U3.34 (GPIO22)
- net UNSKIP: now also SW4.2
- net VOLUME+: now reaches U3.35 (GPIO23)
- net VOLUME+: now also SW2.2
- net SKIP: now reaches U3.36 (GPIO24)
- net SKIP: now also SW5.2
- net CH572_SCK: now reaches U3.4 (GPIO2)
- net CH572_SCK: now also TP13.1
- net at U3.46 (VREG_AVDD): now also C28.2, R16.1
- net at U3.48 (VREG_LX): now also L1.2
- net CH572_MOSI: now reaches U3.5 (GPIO3)
- net CH572_MOSI: now also U10.16 (PA7/MOSI/T4/PWM1/TMR/RST_/CP1), TP11.1
- net at U3.51 (USB_DM): now also R17.2
- net at U3.52 (USB_DP): now also R18.2
- net at U3.60 (QSPI_SS): now also R15.1
- net SD_DETECT: now reaches U3.8 (GPIO5)
- net SD_DETECT: now also Card1.CD, TP9.1
- net SD_EN: now reaches U3.9 (GPIO6)
- net SD_EN: now also Q2.1 (G), R5.2
- net BATTERY+: now reaches CN1.1, Q1.3 (D), R4.2, U5.3 (BAT)
- net BATTERY+: now also C16.1, TP33.1
- net at Card1.1 (DAT2): now also R6.2
- net at Card1.4 (VDD): now also C18.1, Q2.3 (D), R6.1, R7.1, TP15.1
- net at Card1.8 (DAT1): now also R7.2
- net CH572_SCREEN_SCL: now reaches U10.1 (PA3/T/R1/SCL2/SCK_/PWM3/CP0)
- net CH572_SCREEN_SCL: now also J3.3 (Pin_3)
- net CH572_SCREEN_SDA: now reaches U10.20 (PA2/R/T1/SDA2/SCS_/PWM2/TMR1/CN)
- net CH572_SCREEN_SDA: now also J3.4 (Pin_4)
- new net: J2.A5 (CC1), R14.1
- new net: C33.2, C37.2, C38.2, C39.2, C40.2, C41.2, C42.2, C43.2
- new net: R19.2, S3.3, S3.4
- new net: J2.B5 (CC2), R13.1
- new net: R15.2, S2.3, S2.4
- new net: R12.1, S1.3, S1.4
- new net LOUT: CN2.4, R8.1
- new net ROUT: CN2.3, R9.1
- new net RP_D+: J2.A6 (DP1), J2.B6 (DP2), R18.1
- new net RP_D-: J2.A7 (DN1), J2.B7 (DN2), R17.1
- no-connect marks 2 -> 21
Other:
- note added: "1.8v"
- note added: "3.3V low noise"
- note added: "3.3v main power unit"
- note added: "BATTERY"
- note added: "BUTTONS"
- note added: "Battery charging/Load share"
- note added: "Boot Button for wireless chip"
- note added: "CH572 Communication Top left"
- note added: "DAC"
- note added: "SD Card"
- note added: "programming for wireless chip"
- note added: "wireless communication with chip antennna"
- moved on the sheet: C1, C10, C11, C12, C13, C14, C15, C2, C6, C8, C9, CN1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
Changed lines of the file:
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@@
 (kicad_sch
-	(version 20250114)
+	(version 20260101)
 	(generator "eeschema")
-	(generator_version "9.0")
+	(generator_version "10.0")
 	(paper "A1")

Commit message: worked on it
Parts:
- added C31: 0.1uF, CHXXX:0402, symbol fab:C_0603
Connections:
- net BATMON: now also C31.1
- net PWR_GND: now also C31.2
- no-connect marks 21 -> 22
Changed lines of the file:
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@@
 (kicad_sch
-	(version 20260101)
+	(version 20260306)
 	(generator "eeschema")
 	(generator_version "10.0")
